File: SafetyLights/AmbientLight-2.brd (EAGLE design)
At the start: 18.8 x 7.4 mm, 11 parts, among them IC1 SWITCHING-REGULATOR-VARIABLE-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, K1 KEYSTONE-BATTERY-HOLDER-2X-AA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, Q1 MOSFET-N-CHANNEL-VISHAY-SI103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

Commit message: Fridge design updated for new materials and dimensions, AmbientLight-2 and Audio-6 updated for manufacturability
Other:
- board text added: "(C) 2015 Kuy Mainwaring"
- board text added: "100kΩ RES 0603"
- board text added: "10uF CAP 0805"
- board text added: "1MΩ RES 0603"
- board text added: "1uF CAP 0603"
- board text added: "4.7uF CAP 0603"
- board text added: "4.7uH IND 1210"
- board text added: "560kΩ RES 0603"
- board text added: "AmbientLight-2"
- board text added: "CHIP"
- board text added: "X"
Changed lines of the file:
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@@
 <grid distance="0.05" unitdist="inch" unit="inch" style="lines" multiple="1" display="no" altdistance="0.005" altunitdist="inch" altunit="inch"/>
 <layers>
-<layer number="1" name="Top" color="4" fill="1" visible="yes" active="yes"/>
+<layer number="1" name="Top" color="4" fill="1" visible="no" active="yes"/>
 <layer number="2" name="Route2" color="1" fill="3" visible="no" active="no"/>
 <layer number="3" name="Route3" color="4" fill="3" visible="no" active="no"/>
 <layer number="14" name="Route14" color="1" fill="6" visible="no" active="no"/>
 <layer number="15" name="Route15" color="4" fill="6" visible="no" active="no"/>
-<layer number="16" name="Bottom" color="1" fill="1" visible="yes" active="yes"/>
-<layer number="17" name="Pads" color="2" fill="1" visible="yes" active="yes"/>
-<layer number="18" name="Vias" color="2" fill="1" visible="yes" active="yes"/>
-<layer number="19" name="Unrouted" color="3" fill="1" visible="yes" active="yes"/>
+<layer number="16" name="Bottom" color="1" fill="1" visible="no" active="yes"/>
+<layer number="17" name="Pads" color="2" fill="1" visible="no" active="yes"/>
+<layer number="18" name="Vias" color="2" fill="1" visible="no" active="yes"/>
+<layer number="19" name="Unrouted" color="3" fill="1" visible="no" active="yes"/>
 <layer number="20" name="Dimension" color="15" fill="1" visible="yes" active="yes"/>
-<layer number="21" name="tPlace" color="15" fill="1" visible="yes" active="yes"/>
-<layer number="22" name="bPlace" color="7" fill="1" visible="yes" active="yes"/>
+<layer number="21" name="tPlace" color="7" fill="1" visible="yes" active="yes"/>
+<layer number="22" name="bPlace" color="7" fill="1" visible="no" active="yes"/>
 <layer number="23" name="tOrigins" color="15" fill="1" visible="yes" active="yes"/>
-<layer number="24" name="bOrigins" color="15" fill="1" visible="yes" active="yes"/>
+<layer number="24" name="bOrigins" color="15" fill="1" visible="no" active="yes"/>
 <layer number="25" name="tNames" color="7" fill="1" visible="no" active="yes"/>
 <layer number="26" name="bNames" color="7" fill="1" visible="no" active="yes"/>
@@
 <layer number="28" name="bValues" color="7" fill="1" visible="no" active="yes"/>
 <layer number="29" name="tStop" color="7" fill="3" visible="yes" active="yes"/>
-<layer number="30" name="bStop" color="7" fill="6" visible="yes" active="yes"/>
+<layer number="30" name="bStop" color="7" fill="6" visible="no" active="yes"/>
 <layer number="31" name="tCream" color="7" fill="4" visible="no" active="yes"/>
 <layer number="32" name="bCream" color="7" fill="5" visible="no" active="yes"/>
@@
 <layer number="43" name="vRestrict" color="2" fill="10" visible="no" active="yes"/>
 <layer number="44" name="Drills" color="7" fill="1" visible="no" active="yes"/>
-<layer number="45" name="Holes" color="7" fill="1" visible="yes" active="yes"/>
+<layer number="45" name="Holes" color="7" fill="1" visible="no" active="yes"/>
 <layer number="46" name="Milling" color="3" fill="1" visible="no" active="yes"/>
 <layer number="47" name="Measures" color="7" fill="1" visible="no" active="yes"/>
@@
 <layer number="50" name="dxf" color="7" fill="1" visible="no" active="no"/>
 <layer number="51" name="tDocu" color="7" fill="1" visible="yes" active="yes"/>
-<layer number="52" name="bDocu" color="7" fill="1" visible="yes" active="yes"/>
+<layer number="52" name="bDocu" color="7" fill="1" visible="no" active="yes"/>
 <layer number="53" name="tGND_GNDA" color="7" fill="9" visible="no" active="no"/>
 <layer number="54" name="bGND_GNDA" color="1" fill="9" visible="no" active="no"/>
@@
 <layer number="98" name="Guide" color="6" fill="1" visible="no" active="no"/>
 <layer number="100" name="Muster" color="7" fill="1" visible="no" active="no"/>
-<layer number="101" name="tBuild" color="7" fill="1" visible="no" active="yes"/>
+<layer number="101" name="tBuild" color="15" fill="1" visible="yes" active="yes"/>
 <layer number="102" name="bBuild" color="7" fill="1" visible="no" active="yes"/>
 <layer number="103" name="tMap" color="7" fill="1" visible="no" active="yes"/>
@@
 <wire x1="17.145" y1="5.588" x2="17.907" y2="5.588" width="0.254" layer="22"/>
 <wire x1="13.081" y1="1.016" x2="14.097" y2="1.016" width="0.254" layer="22"/>
-<text x="0" y="8.89" size="0.3048" layer="51">https://docs.google.com/spreadsheets/d/1b9Oirg_7CsMoOT67FXmkAzQT9mrNKB5ivZXDMmT1TtM/edit#gid=0</text>
+<text x="0" y="11.43" size="0.3048" layer="51">https://docs.google.com/spreadsheets/d/1b9Oirg_7CsMoOT67FXmkAzQT9mrNKB5ivZXDMmT1TtM/edit#gid=0</text>
+<text x="11.43" y="-2.413" size="1.016" layer="101" font="vector" ratio="15">4.7uH IND 1210</text>
+<text x="6.35" y="-2.921" size="1.016" layer="101" font="vector" ratio="15" rot="R180">4.7uF CAP 0603</text>
+<text x="5.08" y="-1.27" size="1.016" layer="101" font="vector" ratio="15" rot="R180">10uF CAP 0805</text>
+<text x="5.08" y="8.89" size="1.016" layer="101" font="vector" ratio="15" rot="R180">560kΩ RES 0603</text>
+<text x="7.112" y="10.668" size="1.016" layer="101" font="vector" ratio="15" rot="R180">1MΩ RES 0603</text>
+<text x="11.049" y="8.255" size="1.016" layer="101" font="vector" ratio="15">CHIP</text>
+<text x="16.51" y="8.89" size="1.016" layer="101" font="vector" ratio="15">100kΩ RES 0603</text>
+<text x="20.32" y="5.08" size="1.016" layer="101" font="vector" ratio="15">1uF CAP 0603</text>
+<circle x="10.414" y="3.81" radius="0.523634375" width="0.4064" layer="101"/>
+<wire x1="13.716" y1="3.937" x2="19.177" y2="3.937" width="0.1524" layer="101"/>
+<wire x1="19.177" y1="3.937" x2="20.066" y2="4.826" width="0.1524" layer="101"/>
+<wire x1="14.986" y1="5.334" x2="14.986" y2="7.366" width="0.1524" layer="101"/>
+<wire x1="14.986" y1="7.366" x2="16.256" y2="8.636" width="0.1524" layer="101"/>
+<wire x1="10.414" y1="5.461" x2="10.414" y2="7.62" width="0.1524" layer="101"/>
+<wire x1="10.414" y1="7.62" x2="10.795" y2="8.001" width="0.1524" layer="101"/>
+<wire x1="7.747" y1="4.953" x2="7.747" y2="8.636" width="0.1524" layer="101"/>
+<wire x1="7.747" y1="8.636" x2="6.985" y2="9.398" width="0.1524" layer="101"/>
+<wire x1="5.969" y1="5.842" x2="5.969" y2="6.731" width="0.1524" layer="101"/>
+<wire x1="5.969" y1="6.731" x2="5.08" y2="7.62" width="0.1524" layer="101"/>
+<wire x1="5.969" y1="3.175" x2="5.969" y2="-0.254" width="0.1524" layer="101"/>
+<wire x1="5.969" y1="-0.254" x2="5.207" y2="-1.016" width="0.1524" layer="101"/>
+<wire x1="7.747" y1="2.667" x2="7.747" y2="-1.524" width="0.1524" layer="101"/>
+<wire x1="7.747" y1="-1.524" x2="6.604" y2="-2.667" width="0.1524" layer="101"/>
+<wire x1="10.922" y1="1.397" x2="10.922" y2="-0.762" width="0.1524" layer="101"/>
+<wire x1="10.922" y1="-0.762" x2="11.303" y2="-1.143" width="0.1524" layer="101"/>
+<text x="1.016" y="5.207" size="1.016" layer="101" font="vector" ratio="15">X</text>
+<text x="12.827" y="5.207" size="1.016" layer="101" font="vector" ratio="15">X</text>
+<text x="1.27" y="15.24" size="1.524" layer="101" font="vector" ratio="15">AmbientLight-2</text>
+<text x="2.413" y="13.843" size="0.762" layer="101" font="vector" ratio="15">(C) 2015 Kuy Mainwaring</text>
 </plain>
 <attributes>
