File: Audio/pcb/Audio-6.brd (EAGLE design)
At the start: 46.1 x 26.7 mm, 89 parts, among them IC1 AMP-AUDIO-CLASS-D-TI-TPA2006A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, IC2 AMP-AUDIO-CLASS-D-TI-TPA2006A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, IC3 DRIVER-RS485-RS422-SN75176-SO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, IC4 LPC13XXFHN33, IC5 LDO-REGULATOR-FIXED-WITH-ENAB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, IC6 AUDIO-DAC-NXP-UDA1334ATS, IC7 SWITCHING-REGULATOR-VARIABLE-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, K1 HEADER-1X01-NO-SILK, K10 SPEAKER-BLOCK, K11 SPEAKER-BLOCK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

Commit message: Fridge design updated for new materials and dimensions, AmbientLight-2 and Audio-6 updated for manufacturability
Parts:
- C25, C31: value 22u -> 22u 25V
- C26, C30: value 22u -> 22u 10V
- C9: value 4.7u -> 1u
- R17: value (none) -> 22k
- R18: value (none) -> 100k
Connections:
- net N$5 renamed D-
- net N$6 renamed D+
Other:
- board text added: "(C) Kuy Mainwaring 2015"
- board text added: "1.5kΩ RES 0603"
- board text added: "100kΩ RES 0603"
- board text added: "100n CAP 0603"
- board text added: "100nF CAP 0603"
- board text added: "100Ω, 220kΩ, 100Ω, 220kΩ RES, 100nF CAP 0603"
- board text added: "10Ω RES 0603"
- board text added: "12MHz CRYSTAL"
- board text added: "1N4148 DIODE SOD323"
- board text added: "1uF CAP 0603"
- board text added: "22kΩ RES 0603"
- board text added: "22uF CAP 1206"
- board text added: "2x 1.5k RES 0603"
- board text added: "2x 10uF CAP 1206"
- board text added: "2x 12pF CAP 0603"
- board text added: "2x 1uF CAP 0603"
- board text added: "2x 22uF CAP 1206"
- board text added: "2x 33Ω RES 0805"
- board text added: "2x 49.9Ω RES 0603"
- board text added: "2x 6.8nF CAP 0603"
- board text added: "2x FERRITE 0603"
- board text added: "3x 22uF CAP 1206"
- board text added: "4x 150kΩ RES 0603"
- board text added: "4x 1uF CAP 0603"
- board text added: "5x 100nF CAP 0603"
- board text added: "6.8kΩ RES 0603"
- board text added: "6.8nF CAP 0603"
- board text added: "HW MOD: 10kΩ 0402 to GND - !SHUTDOWN! pull-down - TX/!RX! pull-down"
- board text added: "PlayaBeats6"

Commit message: Updates to ambient audio etc.
Connections:
- net N$18 renamed IO3
- net N$8 renamed IO1
- net N$9 renamed IO2
Changed lines of the file:
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@@
 <grid distance="0.05" unitdist="inch" unit="inch" style="lines" multiple="1" display="no" altdistance="0.005" altunitdist="inch" altunit="inch"/>
 <layers>
-<layer number="1" name="Top" color="4" fill="1" visible="no" active="yes"/>
+<layer number="1" name="Top" color="4" fill="1" visible="yes" active="yes"/>
 <layer number="2" name="Route2" color="1" fill="3" visible="no" active="no"/>
 <layer number="3" name="Route3" color="4" fill="3" visible="no" active="no"/>
@@
 <layer number="15" name="Route15" color="4" fill="6" visible="no" active="no"/>
 <layer number="16" name="Bottom" color="1" fill="1" visible="no" active="yes"/>
-<layer number="17" name="Pads" color="2" fill="1" visible="no" active="yes"/>
-<layer number="18" name="Vias" color="2" fill="1" visible="no" active="yes"/>
+<layer number="17" name="Pads" color="2" fill="1" visible="yes" active="yes"/>
+<layer number="18" name="Vias" color="2" fill="1" visible="yes" active="yes"/>
 <layer number="19" name="Unrouted" color="3" fill="1" visible="no" active="yes"/>
 <layer number="20" name="Dimension" color="15" fill="1" visible="yes" active="yes"/>
@@
 <wire x1="15.505" y1="11.405" x2="15.505" y2="10.784" width="0.2032" layer="1"/>
 </signal>
-<signal name="N$8">
+<signal name="IO1">
 <contactref element="IC4" pad="23"/>
 <contactref element="K5" pad="P$1"/>
@@
 <wire x1="21.743" y1="16.23" x2="22.352" y2="15.621" width="0.254" layer="1"/>
 </signal>
-<signal name="N$9">
+<signal name="IO2">
 <contactref element="IC4" pad="24"/>
 <contactref element="K6" pad="P$1"/>
@@
 <wire x1="22.214" y1="16.88" x2="22.352" y2="17.018" width="0.254" layer="1"/>
 </signal>
-<signal name="N$18">
+<signal name="IO3">
 <contactref element="IC4" pad="25"/>
 <contactref element="K14" pad="P$1"/>
