File: Audio/pcb/Audio-6.sch (EAGLE design)
At the start: 89 parts, among them IC1 AMP-AUDIO-CLASS-D-TI-TPA2006A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, IC2 AMP-AUDIO-CLASS-D-TI-TPA2006A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, IC3 DRIVER-RS485-RS422-SN75176-SO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, IC4 LPC13XXFHN33, IC5 LDO-REGULATOR-FIXED-WITH-ENAB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, IC6 AUDIO-DAC-NXP-UDA1334ATS, IC7 SWITCHING-REGULATOR-VARIABLE-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, K1 HEADER-1X01-NO-SILK, K10 SPEAKER-BLOCK, K11 SPEAKER-BLOCK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

Commit message: Fridge design updated for new materials and dimensions, AmbientLight-2 and Audio-6 updated for manufacturability
Parts:
- C25, C31: value 22u -> 22u 25V
- C26, C30: value 22u -> 22u 10V
- C9: value 4.7u -> 1u
- R17: value (none) -> 22k
- R18: value (none) -> 100k
Connections:
- net N$5 renamed D-
- net N$6 renamed D+
Changed lines of the file:
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@@
 <part name="C7" library="Outbreak" deviceset="CAP" device="-0603-MIN" value="100n"/>
 <part name="C8" library="Outbreak" deviceset="CAP" device="-0603-MIN" value="100n"/>
-<part name="C9" library="Outbreak" deviceset="CAP" device="-0603-MIN" value="4.7u"/>
+<part name="C9" library="Outbreak" deviceset="CAP" device="-0603-MIN" value="1u"/>
 <part name="GND12" library="Outbreak" deviceset="GND" device=""/>
 <part name="GND13" library="Outbreak" deviceset="GND" device=""/>
@@
 <part name="L1" library="Outbreak" deviceset="INDUCTOR" device="-6X6MM" value="10u"/>
 <part name="C29" library="Outbreak" deviceset="CAP" device="-0603-MIN" value="10n"/>
-<part name="C30" library="Outbreak" deviceset="CAP" device="-1206" value="22u"/>
-<part name="C31" library="Outbreak" deviceset="CAP" device="-1206" value="22u"/>
+<part name="C30" library="Outbreak" deviceset="CAP" device="-1206" value="22u 10V"/>
+<part name="C31" library="Outbreak" deviceset="CAP" device="-1206" value="22u 25V"/>
 <part name="C32" library="Outbreak" deviceset="CAP" device="-0603-MIN" value="100n"/>
 <part name="C33" library="Outbreak" deviceset="CAP" device="-0603-MIN" value="6.8n"/>
 <part name="R16" library="Outbreak" deviceset="RESISTOR" device="-0603-MIN" value="6.8k"/>
-<part name="R17" library="Outbreak" deviceset="RESISTOR" device="-0603-MIN"/>
-<part name="R18" library="Outbreak" deviceset="RESISTOR" device="-0603-MIN"/>
+<part name="R17" library="Outbreak" deviceset="RESISTOR" device="-0603-MIN" value="22k"/>
+<part name="R18" library="Outbreak" deviceset="RESISTOR" device="-0603-MIN" value="100k"/>
 <part name="V12" library="Outbreak" deviceset="V" device=""/>
 <part name="V13" library="Outbreak" deviceset="V" device=""/>
@@
 <part name="K10" library="BMan" deviceset="SPEAKER-BLOCK" device=""/>
 <part name="K11" library="BMan" deviceset="SPEAKER-BLOCK" device=""/>
-<part name="C25" library="Outbreak" deviceset="CAP" device="-1206" value="22u"/>
+<part name="C25" library="Outbreak" deviceset="CAP" device="-1206" value="22u 25V"/>
 <part name="R23" library="Outbreak" deviceset="RESISTOR" device="-0603-MIN" value="100k"/>
 <part name="K8" library="Outbreak" deviceset="USB-5-PIN" device="-MICROB-FCI-10118193-NARROW"/>
@@
 <part name="K12" library="Outbreak" deviceset="HEADER-1X01" device="-NO-SILK"/>
 <part name="K13" library="Outbreak" deviceset="HEADER-1X01" device="-NO-SILK"/>
-<part name="C26" library="Outbreak" deviceset="CAP" device="-1206" value="22u"/>
+<part name="C26" library="Outbreak" deviceset="CAP" device="-1206" value="22u 10V"/>
 <part name="D1" library="Outbreak" deviceset="DIODE" device="-SOD323"/>
 <part name="U1" library="Outbreak" deviceset="GND-ISOLATOR" device="-0.032&quot;"/>
@@
 </segment>
 </net>
-<net name="N$5" class="0">
+<net name="D-" class="0">
 <segment>
 <pinref part="IC4" gate="G$1" pin="PIO3_4/USB_D-"/>
@@
 </segment>
 </net>
-<net name="N$6" class="0">
+<net name="D+" class="0">
 <segment>
 <pinref part="IC4" gate="G$1" pin="PIO3_5/USB_D+"/>

Commit message: Updates to ambient audio etc.
Connections:
- net N$18 renamed IO3
- net N$8 renamed IO1
- net N$9 renamed IO2
Changed lines of the file:
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@@
 </segment>
 </net>
-<net name="N$8" class="0">
+<net name="IO1" class="0">
 <segment>
 <pinref part="IC4" gate="G$1" pin="TDO/PIO1_1/AD2/CT32B1_MAT0"/>
@@
 </segment>
 </net>
-<net name="N$9" class="0">
+<net name="IO2" class="0">
 <segment>
 <pinref part="IC4" gate="G$1" pin="TRST/PIO1_2/AD3/CT32B1_MAT1"/>
@@
 </segment>
 </net>
-<net name="N$18" class="0">
+<net name="IO3" class="0">
 <segment>
 <pinref part="IC4" gate="G$1" pin="SWDIO/PIO1_3/AD4/CT32B1_MAT2"/>
