File: Fridge/Fridge31-1.sch (EAGLE design)
At the start: 0 parts

Commit message: Fridge design updated for new materials and dimensions, AmbientLight-2 and Audio-6 updated for manufacturability
Other:
- note added: "*omit for lid"
- note added: "0.2" thick plywood"
- note added: "0.75x1.5" stud"
- note added: "1.5x1.5" stud"
- note added: "Supercooler XY (bottom, lid*)"
- note added: "Supercooler XY (cross section)"
- note added: "Supercooler XY (top below lid)"
- note added: "UP"
- note added: "X"
- note added: "b"
- note added: "b*"
- note added: "external height=24" internal hight=20""
- note removed: "0.5" thick OSB"
- note removed: "1x1" stud"
- note removed: "Burning Man 31 Supercooler Assembly"

Commit message: Updates to ambient audio etc.
Other:
- note added: "20.20""
- note added: "23.20""
- note added: "25.50""
- note added: "32.60""
- note added: "Supercooler XZ (side cross-section)"
- note added: "Z"
